File: Sensors/SERIS/Solar_Irradiance_Sensor.brd (EAGLE design)
At the start: 100 x 80 mm, 8 parts, among them IC1 LM324N

Commit message: .
Parts:
- moved JP1 5.24 mm to (57.1, 24.1)
- moved C1 4.02 mm to (44.5, 50.8)
- turned JP4 to 180 degrees
Connections:
- removed net N$3: C1.1, IC1.3, R1.2
- new net N$2: C1.1, IC1.3, R1.2, U$1.S18
Changed lines of the file:
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@@
 <elements>
 <element name="IC1" library="linear" package="DIL14" value="LM324N" x="33.02" y="48.26" rot="R90"/>
-<element name="JP1" library="SparkFun-Connectors" package="1X02_2.54_SCREWTERM" value="M022.54MM_SCREWTERM" x="52.07" y="25.4"/>
+<element name="JP1" library="SparkFun-Connectors" package="1X02_2.54_SCREWTERM" value="M022.54MM_SCREWTERM" x="57.15" y="24.13"/>
 <element name="U$1" library="wasp" package="WASP" value="WASP" x="50.8" y="54.61"/>
 <element name="R1" library="rcl" package="0207/10" value="100k" x="55.88" y="35.56" rot="R90"/>
 <element name="R2" library="rcl" package="0207/10" value="100k" x="43.18" y="35.56" rot="R270"/>
 <element name="R3" library="rcl" package="0207/10" value="2k" x="49.53" y="35.56" rot="R90"/>
-<element name="C1" library="rcl" package="C025-024X044" value="0.1uF" x="43.18" y="46.99" rot="R90"/>
-<element name="JP4" library="pinhead" package="2X06" value="MAX31865" x="39.37" y="67.31"/>
+<element name="C1" library="rcl" package="C025-024X044" value="0.1uF" x="44.45" y="50.8" rot="R90"/>
+<element name="JP4" library="pinhead" package="2X06" value="MAX31865" x="39.37" y="67.31" rot="R180"/>
 </elements>
 <signals>
@@
 <contactref element="JP4" pad="10"/>
 <contactref element="JP1" pad="P2"/>
-<wire x1="43.18" y1="66.04" x2="60.96" y2="57.15" width="0" layer="19" extent="1-1"/>
-<wire x1="43.18" y1="68.58" x2="43.18" y2="66.04" width="0" layer="19" extent="1-1"/>
-<wire x1="43.18" y1="48.26" x2="43.18" y2="66.04" width="0" layer="19" extent="1-1"/>
-<wire x1="29.21" y1="48.26" x2="43.18" y2="48.26" width="0" layer="19" extent="1-1"/>
-<wire x1="20.32" y1="64.77" x2="29.21" y2="48.26" width="0" layer="19" extent="1-1"/>
-<wire x1="49.53" y1="30.48" x2="43.18" y2="48.26" width="0" layer="19" extent="1-1"/>
-<wire x1="52.07" y1="25.4" x2="49.53" y2="30.48" width="0" layer="19" extent="1-1"/>
+<wire x1="44.45" y1="52.07" x2="60.96" y2="57.15" width="0" layer="19" extent="1-1"/>
+<wire x1="29.21" y1="48.26" x2="44.45" y2="52.07" width="0" layer="19" extent="1-1"/>
+<wire x1="35.56" y1="66.04" x2="44.45" y2="52.07" width="0" layer="19" extent="1-1"/>
+<wire x1="35.56" y1="68.58" x2="35.56" y2="66.04" width="0" layer="19" extent="1-1"/>
+<wire x1="20.32" y1="64.77" x2="35.56" y2="66.04" width="0" layer="19" extent="1-1"/>
+<wire x1="49.53" y1="30.48" x2="44.45" y2="52.07" width="0" layer="19" extent="1-1"/>
+<wire x1="57.15" y1="24.13" x2="49.53" y2="30.48" width="0" layer="19" extent="1-1"/>
 </signal>
 <signal name="N$1">
@@
 <wire x1="43.18" y1="40.64" x2="49.53" y2="40.64" width="0" layer="19" extent="1-1"/>
 <wire x1="36.83" y1="43.18" x2="43.18" y2="40.64" width="0" layer="19" extent="1-1"/>
-</signal>
-<signal name="N$3">
-<contactref element="R1" pad="2"/>
-<contactref element="IC1" pad="3"/>
-<contactref element="C1" pad="1"/>
-<wire x1="43.18" y1="45.72" x2="55.88" y2="40.64" width="0" layer="19" extent="1-1"/>
-<wire x1="36.83" y1="45.72" x2="43.18" y2="45.72" width="0" layer="19" extent="1-1"/>
 </signal>
 <signal name="SOLAR_OUTPUT">
@@
 <contactref element="JP4" pad="11"/>
 <contactref element="JP4" pad="12"/>
-<wire x1="45.72" y1="66.04" x2="45.72" y2="68.58" width="0" layer="19" extent="1-1"/>
-<wire x1="36.83" y1="48.26" x2="45.72" y2="66.04" width="0" layer="19" extent="1-1"/>
+<wire x1="33.02" y1="66.04" x2="33.02" y2="68.58" width="0" layer="19" extent="1-1"/>
+<wire x1="36.83" y1="48.26" x2="33.02" y2="66.04" width="0" layer="19" extent="1-1"/>
 <wire x1="20.32" y1="41.91" x2="36.83" y2="48.26" width="0" layer="19" extent="1-1"/>
 </signal>
@@
 <contactref element="R1" pad="1"/>
 <contactref element="JP1" pad="P1"/>
-<wire x1="54.61" y1="25.4" x2="55.88" y2="30.48" width="0" layer="19" extent="1-1"/>
+<wire x1="59.69" y1="24.13" x2="55.88" y2="30.48" width="0" layer="19" extent="1-1"/>
 </signal>
 <signal name="INT">
@@
 <contactref element="JP4" pad="8"/>
 <contactref element="U$1" pad="A7"/>
-<wire x1="40.64" y1="68.58" x2="60.96" y2="54.61" width="0" layer="19" extent="1-1"/>
+<wire x1="38.1" y1="66.04" x2="60.96" y2="54.61" width="0" layer="19" extent="1-1"/>
 </signal>
 <signal name="MISO">
 <contactref element="JP4" pad="6"/>
 <contactref element="U$1" pad="A12"/>
-<wire x1="60.96" y1="41.91" x2="38.1" y2="68.58" width="0" layer="19" extent="1-1"/>
+<wire x1="60.96" y1="41.91" x2="40.64" y2="66.04" width="0" layer="19" extent="1-1"/>
 </signal>
 <signal name="MOSI">
 <contactref element="U$1" pad="A11"/>
 <contactref element="JP4" pad="4"/>
-<wire x1="35.56" y1="68.58" x2="60.96" y2="44.45" width="0" layer="19" extent="1-1"/>
+<wire x1="60.96" y1="44.45" x2="43.18" y2="66.04" width="0" layer="19" extent="1-1"/>
 </signal>
 <signal name="SS">
 <contactref element="JP4" pad="2"/>
 <contactref element="U$1" pad="S12"/>
-<wire x1="20.32" y1="54.61" x2="33.02" y2="68.58" width="0" layer="19" extent="1-1"/>
+<wire x1="20.32" y1="54.61" x2="45.72" y2="66.04" width="0" layer="19" extent="1-1"/>
+</signal>
+<signal name="N$2">
+<contactref element="R1" pad="2"/>
+<contactref element="IC1" pad="3"/>
+<contactref element="C1" pad="1"/>
+<contactref element="U$1" pad="S18"/>
+<wire x1="44.45" y1="49.53" x2="55.88" y2="40.64" width="0" layer="19" extent="1-1"/>
+<wire x1="36.83" y1="45.72" x2="44.45" y2="49.53" width="0" layer="19" extent="1-1"/>
+<wire x1="20.32" y1="46.99" x2="36.83" y2="45.72" width="0" layer="19" extent="1-1"/>
 </signal>
 </signals>

Commit message: updated SERIS project
Parts:
- moved JP1 10.2 mm to (67.3, 25.4)
- moved JP4 1.27 mm to (38.1, 67.3)
Changed lines of the file:
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@@
 <elements>
 <element name="IC1" library="linear" package="DIL14" value="LM324N" x="33.02" y="48.26" rot="R90"/>
-<element name="JP1" library="SparkFun-Connectors" package="1X02_2.54_SCREWTERM" value="M022.54MM_SCREWTERM" x="57.15" y="24.13"/>
+<element name="JP1" library="SparkFun-Connectors" package="1X02_2.54_SCREWTERM" value="M022.54MM_SCREWTERM" x="67.31" y="25.4"/>
 <element name="U$1" library="wasp" package="WASP" value="WASP" x="50.8" y="54.61"/>
 <element name="R1" library="rcl" package="0207/10" value="100k" x="55.88" y="35.56" rot="R90"/>
@@
 <element name="R3" library="rcl" package="0207/10" value="2k" x="49.53" y="35.56" rot="R90"/>
 <element name="C1" library="rcl" package="C025-024X044" value="0.1uF" x="44.45" y="50.8" rot="R90"/>
-<element name="JP4" library="pinhead" package="2X06" value="MAX31865" x="39.37" y="67.31" rot="R180"/>
+<element name="JP4" library="pinhead" package="2X06" value="MAX31865" x="38.1" y="67.31" rot="R180"/>
 </elements>
 <signals>
@@
 <wire x1="44.45" y1="52.07" x2="60.96" y2="57.15" width="0" layer="19" extent="1-1"/>
 <wire x1="29.21" y1="48.26" x2="44.45" y2="52.07" width="0" layer="19" extent="1-1"/>
-<wire x1="35.56" y1="66.04" x2="44.45" y2="52.07" width="0" layer="19" extent="1-1"/>
-<wire x1="35.56" y1="68.58" x2="35.56" y2="66.04" width="0" layer="19" extent="1-1"/>
-<wire x1="20.32" y1="64.77" x2="35.56" y2="66.04" width="0" layer="19" extent="1-1"/>
+<wire x1="34.29" y1="66.04" x2="44.45" y2="52.07" width="0" layer="19" extent="1-1"/>
+<wire x1="34.29" y1="68.58" x2="34.29" y2="66.04" width="0" layer="19" extent="1-1"/>
+<wire x1="20.32" y1="64.77" x2="34.29" y2="66.04" width="0" layer="19" extent="1-1"/>
 <wire x1="49.53" y1="30.48" x2="44.45" y2="52.07" width="0" layer="19" extent="1-1"/>
-<wire x1="57.15" y1="24.13" x2="49.53" y2="30.48" width="0" layer="19" extent="1-1"/>
+<wire x1="67.31" y1="25.4" x2="49.53" y2="30.48" width="0" layer="19" extent="1-1"/>
 </signal>
 <signal name="N$1">
@@
 <contactref element="JP4" pad="11"/>
 <contactref element="JP4" pad="12"/>
-<wire x1="33.02" y1="66.04" x2="33.02" y2="68.58" width="0" layer="19" extent="1-1"/>
-<wire x1="36.83" y1="48.26" x2="33.02" y2="66.04" width="0" layer="19" extent="1-1"/>
+<wire x1="31.75" y1="66.04" x2="31.75" y2="68.58" width="0" layer="19" extent="1-1"/>
+<wire x1="36.83" y1="48.26" x2="31.75" y2="66.04" width="0" layer="19" extent="1-1"/>
 <wire x1="20.32" y1="41.91" x2="36.83" y2="48.26" width="0" layer="19" extent="1-1"/>
 </signal>
@@
 <contactref element="R1" pad="1"/>
 <contactref element="JP1" pad="P1"/>
-<wire x1="59.69" y1="24.13" x2="55.88" y2="30.48" width="0" layer="19" extent="1-1"/>
+<wire x1="55.88" y1="30.48" x2="69.85" y2="25.4" width="0" layer="19" extent="1-1"/>
 </signal>
 <signal name="INT">
@@
 <contactref element="JP4" pad="8"/>
 <contactref element="U$1" pad="A7"/>
-<wire x1="38.1" y1="66.04" x2="60.96" y2="54.61" width="0" layer="19" extent="1-1"/>
+<wire x1="36.83" y1="66.04" x2="60.96" y2="54.61" width="0" layer="19" extent="1-1"/>
 </signal>
 <signal name="MISO">
 <contactref element="JP4" pad="6"/>
 <contactref element="U$1" pad="A12"/>
-<wire x1="60.96" y1="41.91" x2="40.64" y2="66.04" width="0" layer="19" extent="1-1"/>
+<wire x1="60.96" y1="41.91" x2="39.37" y2="66.04" width="0" layer="19" extent="1-1"/>
 </signal>
 <signal name="MOSI">
 <contactref element="U$1" pad="A11"/>
 <contactref element="JP4" pad="4"/>
-<wire x1="60.96" y1="44.45" x2="43.18" y2="66.04" width="0" layer="19" extent="1-1"/>
+<wire x1="60.96" y1="44.45" x2="41.91" y2="66.04" width="0" layer="19" extent="1-1"/>
 </signal>
 <signal name="SS">
 <contactref element="JP4" pad="2"/>
 <contactref element="U$1" pad="S12"/>
-<wire x1="20.32" y1="54.61" x2="45.72" y2="66.04" width="0" layer="19" extent="1-1"/>
+<wire x1="20.32" y1="54.61" x2="44.45" y2="66.04" width="0" layer="19" extent="1-1"/>
 </signal>
 <signal name="N$2">
